File: motors.sch (KiCad schematic (older format))
At the start: 24 parts, among them M1 ALIS-CUSTOM-PARTS_POWERPADS, M2 ALIS-CUSTOM-PARTS_POWERPADS, M3 ALIS-CUSTOM-PARTS_POWERPADS, M4 ALIS-CUSTOM-PARTS_POWERPADS, M5 ALIS-CUSTOM-PARTS_POWERPADS, Q2 BSS138, Q3 BSS138, Q4 BSS138, Q5 BSS138, Q6 BSS138

Commit message: added lots of stuff
Parts:
- D6, D7, D8, D9: footprint Diodes_SMD:SMA_Standard -> Diodes_SMD:SOD-323
Changed lines of the file:
@@
 EESchema Schematic File Version 2
+LIBS:stm32f4_lqfp64_mpu6050-rescue
 LIBS:power
 LIBS:device
@@
 LIBS:minimal
 LIBS:alis_parts
+LIBS:sensors
+LIBS:stm32
 LIBS:stm32f4_lqfp64_mpu6050-cache
 EELAYER 25 0
@@
 $Descr A4 11693 8268
 encoding utf-8
-Sheet 3 7
+Sheet 3 10
 Title ""
 Date ""
@@
 BUZZER
 $Comp
-L GND #PWR14
+L GND #PWR21
 U 1 1 569BDE16
 P 8200 3350
-F 0 "#PWR14" H 8200 3100 50  0001 C CNN
+F 0 "#PWR21" H 8200 3100 50  0001 C CNN
 F 1 "GND" H 8208 3176 50  0000 C CNN
 F 2 "" H 8200 3350 50  0000 C CNN
@@
 F 0 "D9" H 6500 3066 50  0000 C CNN
 F 1 "D" H 6500 2974 50  0000 C CNN
-F 2 "Diodes_SMD:SMA_Standard" H 6500 2850 50  0001 C CNN
+F 2 "Diodes_SMD:SOD-323" H 6500 2850 50  0001 C CNN
 F 3 "" H 6500 2850 50  0000 C CNN
 	1    6500 2850
@@
 $EndComp
 $Comp
-L GND #PWR13
+L GND #PWR19
 U 1 1 569BDE42
 P 6750 3350
-F 0 "#PWR13" H 6750 3100 50  0001 C CNN
+F 0 "#PWR19" H 6750 3100 50  0001 C CNN
 F 1 "GND" H 6758 3176 50  0000 C CNN
 F 2 "" H 6750 3350 50  0000 C CNN
@@
 PWM3
 $Comp
-L GND #PWR10
+L GND #PWR16
 U 1 1 569BDE75
 P 3150 3350
-F 0 "#PWR10" H 3150 3100 50  0001 C CNN
+F 0 "#PWR16" H 3150 3100 50  0001 C CNN
 F 1 "GND" H 3158 3176 50  0000 C CNN
 F 2 "" H 3150 3350 50  0000 C CNN
@@
 PWM4
 $Comp
-L GND #PWR11
+L GND #PWR17
 U 1 1 569BDE8A
 P 4350 3350
-F 0 "#PWR11" H 4350 3100 50  0001 C CNN
+F 0 "#PWR17" H 4350 3100 50  0001 C CNN
 F 1 "GND" H 4358 3176 50  0000 C CNN
 F 2 "" H 4350 3350 50  0000 C CNN
@@
 $EndComp
 $Comp
-L GND #PWR12
+L GND #PWR18
 U 1 1 569BDE90
 P 5550 3350
-F 0 "#PWR12" H 5550 3100 50  0001 C CNN
+F 0 "#PWR18" H 5550 3100 50  0001 C CNN
 F 1 "GND" H 5558 3176 50  0000 C CNN
 F 2 "" H 5550 3350 50  0000 C CNN
@@
 F 0 "D8" H 5300 3066 50  0000 C CNN
 F 1 "D" H 5300 2974 50  0000 C CNN
-F 2 "Diodes_SMD:SMA_Standard" H 5300 2850 50  0001 C CNN
+F 2 "Diodes_SMD:SOD-323" H 5300 2850 50  0001 C CNN
 F 3 "" H 5300 2850 50  0000 C CNN
 	1    5300 2850
@@
 F 0 "D6" H 2900 3066 50  0000 C CNN
 F 1 "D" H 2900 2974 50  0000 C CNN
-F 2 "Diodes_SMD:SMA_Standard" H 2900 2850 50  0001 C CNN
+F 2 "Diodes_SMD:SOD-323" H 2900 2850 50  0001 C CNN
 F 3 "" H 2900 2850 50  0000 C CNN
 	1    2900 2850
@@
 F 0 "D7" H 4100 3066 50  0000 C CNN
 F 1 "D" H 4100 2974 50  0000 C CNN
-F 2 "Diodes_SMD:SMA_Standard" H 4100 2850 50  0001 C CNN
+F 2 "Diodes_SMD:SOD-323" H 4100 2850 50  0001 C CNN
 F 3 "" H 4100 2850 50  0000 C CNN
 	1    4100 2850
@@
 VCC
 $Comp
-L GND #PWR9
+L GND #PWR2
 U 1 1 569BFFAD
 P 1200 1500
-F 0 "#PWR9" H 1200 1250 50  0001 C CNN
+F 0 "#PWR2" H 1200 1250 50  0001 C CNN
 F 1 "GND" H 1208 1326 50  0000 C CNN
 F 2 "" H 1200 1500 50  0000 C CNN
